Commit message: kobuki platform VLP-16 fix + xacro samples

File: ros/kinetic/ubuntu/xenial/desktop-full-turtlebot/config/samples/turtlebot_description/robots/kobuki_hexagons_VLP-16.urdf.xacro (robot description, xacro)
@@ -12,7 +12,4 @@
   <kobuki/>
   <stack_hexagons parent="base_link"/>
-  <!--<VLP-16 parent="base_link" name="velodyne" topic="/velodyne_points" hz="10" samples="440">-->
-  <VLP-16 parent="base_link" name="velodyne" topic="/velodyne_points" hz="10" samples="1875">
-    <origin xyz="0 0 0.4" rpy="0 0 0" />
-  </VLP-16>
+  <VLP-16 parent="VLP=16_base_link"/>
 </robot>

File: ros/kinetic/ubuntu/xenial/desktop-full-turtlebot/config/samples/turtlebot_description/robots/kobuki_hexagons_astra.urdf.xacro (robot description, xacro)
@@ -3,5 +3,5 @@
     - Base      : kobuki
     - Stacks    : hexagons
-    - 3d Sensor : VLP-16
+    - 3d Sensor : astra
 -->
 <robot name="turtlebot" xmlns:xacro="http://ros.org/wiki/xacro">
@@ -9,10 +9,7 @@
   <xacro:include filename="$(find kobuki_description)/urdf/kobuki.urdf.xacro" />
   <xacro:include filename="$(find turtlebot_description)/urdf/stacks/hexagons.urdf.xacro"/>
-  <xacro:include filename="$(find velodyne_description)/urdf/VLP-16.urdf.xacro"/>
+  <xacro:include filename="$(find turtlebot_description)/urdf/sensors/astra.urdf.xacro"/>
   <kobuki/>
   <stack_hexagons parent="base_link"/>
-  <!--<VLP-16 parent="base_link" name="velodyne" topic="/velodyne_points" hz="10" samples="440">-->
-  <VLP-16 parent="base_link" name="velodyne" topic="/velodyne_points" hz="10" samples="1875">
-    <origin xyz="0 0 0.4" rpy="0 0 0" />
-  </VLP-16>
+  <sensor_astra parent="base_link"/>
 </robot>

File: ros/kinetic/ubuntu/xenial/desktop-full-turtlebot/config/samples/turtlebot_description/robots/kobuki_hexagons_asus_xtion_pro.urdf.xacro (robot description, xacro)
@@ -3,5 +3,5 @@
     - Base      : kobuki
     - Stacks    : hexagons
-    - 3d Sensor : VLP-16
+    - 3d Sensor : kinect
 -->
 <robot name="turtlebot" xmlns:xacro="http://ros.org/wiki/xacro">
@@ -9,10 +9,7 @@
   <xacro:include filename="$(find kobuki_description)/urdf/kobuki.urdf.xacro" />
   <xacro:include filename="$(find turtlebot_description)/urdf/stacks/hexagons.urdf.xacro"/>
-  <xacro:include filename="$(find velodyne_description)/urdf/VLP-16.urdf.xacro"/>
+  <xacro:include filename="$(find turtlebot_description)/urdf/sensors/asus_xtion_pro.urdf.xacro"/>
   <kobuki/>
-  <stack_hexagons parent="base_link"/>
-  <!--<VLP-16 parent="base_link" name="velodyne" topic="/velodyne_points" hz="10" samples="440">-->
-  <VLP-16 parent="base_link" name="velodyne" topic="/velodyne_points" hz="10" samples="1875">
-    <origin xyz="0 0 0.4" rpy="0 0 0" />
-  </VLP-16>
+  <stack_hexagons                 parent="base_link"/>
+  <sensor_asus_xtion_pro          parent="base_link"/>
 </robot>

File: ros/kinetic/ubuntu/xenial/desktop-full-turtlebot/config/samples/turtlebot_description/robots/kobuki_hexagons_asus_xtion_pro_offset.urdf.xacro (robot description, xacro)
@@ -3,5 +3,5 @@
     - Base      : kobuki
     - Stacks    : hexagons
-    - 3d Sensor : VLP-16
+    - 3d Sensor : kinect
 -->
 <robot name="turtlebot" xmlns:xacro="http://ros.org/wiki/xacro">
@@ -9,10 +9,7 @@
   <xacro:include filename="$(find kobuki_description)/urdf/kobuki.urdf.xacro" />
   <xacro:include filename="$(find turtlebot_description)/urdf/stacks/hexagons.urdf.xacro"/>
-  <xacro:include filename="$(find velodyne_description)/urdf/VLP-16.urdf.xacro"/>
+  <xacro:include filename="$(find turtlebot_description)/urdf/sensors/asus_xtion_pro_offset.urdf.xacro"/>
   <kobuki/>
-  <stack_hexagons parent="base_link"/>
-  <!--<VLP-16 parent="base_link" name="velodyne" topic="/velodyne_points" hz="10" samples="440">-->
-  <VLP-16 parent="base_link" name="velodyne" topic="/velodyne_points" hz="10" samples="1875">
-    <origin xyz="0 0 0.4" rpy="0 0 0" />
-  </VLP-16>
+  <stack_hexagons                 parent="base_link"/>
+  <sensor_asus_xtion_pro_offset   parent="base_link"/>
 </robot>

File: ros/kinetic/ubuntu/xenial/desktop-full-turtlebot/config/samples/turtlebot_description/robots/kobuki_hexagons_kinect.urdf.xacro (robot description, xacro)
@@ -3,5 +3,5 @@
     - Base      : kobuki
     - Stacks    : hexagons
-    - 3d Sensor : VLP-16
+    - 3d Sensor : kinect
 -->
 <robot name="turtlebot" xmlns:xacro="http://ros.org/wiki/xacro">
@@ -9,10 +9,7 @@
   <xacro:include filename="$(find kobuki_description)/urdf/kobuki.urdf.xacro" />
   <xacro:include filename="$(find turtlebot_description)/urdf/stacks/hexagons.urdf.xacro"/>
-  <xacro:include filename="$(find velodyne_description)/urdf/VLP-16.urdf.xacro"/>
+  <xacro:include filename="$(find turtlebot_description)/urdf/sensors/kinect.urdf.xacro"/>
   <kobuki/>
   <stack_hexagons parent="base_link"/>
-  <!--<VLP-16 parent="base_link" name="velodyne" topic="/velodyne_points" hz="10" samples="440">-->
-  <VLP-16 parent="base_link" name="velodyne" topic="/velodyne_points" hz="10" samples="1875">
-    <origin xyz="0 0 0.4" rpy="0 0 0" />
-  </VLP-16>
+  <sensor_kinect  parent="base_link"/>
 </robot>

File: ros/kinetic/ubuntu/xenial/desktop-full-turtlebot/config/samples/turtlebot_description/robots/kobuki_hexagons_r200.urdf.xacro (robot description, xacro)
@@ -3,5 +3,5 @@
     - Base      : kobuki
     - Stacks    : hexagons
-    - 3d Sensor : VLP-16
+    - 3d Sensor : r200
 -->
 <robot name="turtlebot" xmlns:xacro="http://ros.org/wiki/xacro">
@@ -9,10 +9,7 @@
   <xacro:include filename="$(find kobuki_description)/urdf/kobuki.urdf.xacro" />
   <xacro:include filename="$(find turtlebot_description)/urdf/stacks/hexagons.urdf.xacro"/>
-  <xacro:include filename="$(find velodyne_description)/urdf/VLP-16.urdf.xacro"/>
+  <xacro:include filename="$(find turtlebot_description)/urdf/sensors/r200.urdf.xacro"/>
   <kobuki/>
   <stack_hexagons parent="base_link"/>
-  <!--<VLP-16 parent="base_link" name="velodyne" topic="/velodyne_points" hz="10" samples="440">-->
-  <VLP-16 parent="base_link" name="velodyne" topic="/velodyne_points" hz="10" samples="1875">
-    <origin xyz="0 0 0.4" rpy="0 0 0" />
-  </VLP-16>
+  <sensor_r200  parent="base_link"/>
 </robot>
